File: PCB/Matrix.kicad_pcb (KiCad board)
At the start: 2 copper layers, 40 x 55 mm, 192 parts, among them J1 USB_C_Receptacle_USB2.0_14P, J2 Conn_01x03_Pin, J3 Conn_01x13_Pin, J4 Conn_01x06_Pin, J5 Conn_01x04_Pin, J6 Conn_01x03_Pin, SW1 Switch, U1 RP2040, U2 NCP1117-3.3_SOT223, U3 W25Q128JVS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

Commit message: Add files via upload
Parts:
- removed R3, R4: 27.4, Resistor_SMD:R_0402_1005Metric
Connections:
- U1 pad 46: Net-(U1-USB_DM) -> D-
- U1 pad 47: Net-(U1-USB_DP) -> D+
Routing:
- net D+: track 22.3 -> 26.4 mm
- net D-: track 21.9 -> 25.7 mm
- net Net-(U1-USB_DM): track 3.45 -> 0.00 mm
- net Net-(U1-USB_DP): track 3.13 -> 0.00 mm
- net Net-(J5-Pin_1): track 29.5 -> 29.0 mm, vias 2 -> 4
- added copper zone on F.Cu, net GND
