File: PCB/Matrix.kicad_pcb (KiCad board)
At the start: 2 copper layers, 40 x 55 mm, 190 parts, among them J1 USB_C_Receptacle_USB2.0_14P, J2 Conn_01x03_Pin, J3 Conn_01x13_Pin, J4 Conn_01x06_Pin, J5 Conn_01x04_Pin, J6 Conn_01x03_Pin, SW1 Switch, U1 RP2040, U2 NCP1117-3.3_SOT223, U3 W25Q128JVS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

Commit message: Add files via upload
Routing:
- added copper zone on B.Cu, net GND
