File: PCB/Matrix.kicad_sch (KiCad schematic)
At the start: 189 parts, among them J1 USB_C_Receptacle_USB2.0_14P, J2 Conn_01x03_Pin, J3 Conn_01x04_Pin, J4 Conn_01x04_Pin, SW1 Switch, U1 RP2040, U2 NCP1117-3.3_SOT223, U3 W25Q128JVS, U4 IS31FL3737, Y1 Crystal_GND24

Commit message: Add files via upload
Parts:
- removed J3, J4: Conn_01x04_Pin, Connector_PinHeader_2.54mm:PinHeader_2x02_P2.54mm_Vertical, symbol Connector:Conn_01x04_Pin
- added J3, J4: Conn_01x11_Pin, Connector_PinHeader_2.54mm:PinHeader_2x06_P2.54mm_Vertical, symbol Connector:Conn_01x11_Pin
- added J6: Conn_01x04_Socket, Connector_PinHeader_2.54mm:PinHeader_1x04_P2.54mm_Vertical, symbol Connector:Conn_01x04_Socket
- C1, C2: footprint Capacitor_SMD:C_0402_1005Metric -> Capacitor_SMD:C_0603_1608Metric
- D1, D10, D100, D101, D102, D103, D104, D105, D106, D107, D108, D109, D11, D110, D111, D112, D113, D114, D115, D116, D117, D118, D119, D12, D120, D121, D122, D123, D124, D125, D126, D127, D128, D129, D13, D130, D131, D132, D133, D134, D135, D136, D137, D138, D139, D14, D140, D141, D142, D143, D144, D15, D16, D17, D18, D19, D2, D20, D21, D22, D23, D24, D25, D26, D27, D28, D29, D3, D30, D31, D32, D33, D34, D35, D36, D37, D38, D39, D4, D40, D41, D42, D43, D44, D45, D46, D47, D48, D49, D5, D50, D51, D52, D53, D54, D55, D56, D57, D58, D59, D6, D60, D61, D62, D63, D64, D65, D66, D67, D68, D69, D7, D70, D71, D72, D73, D74, D75, D76, D77, D78, D79, D8, D80, D81, D82, D83, D84, D85, D86, D87, D88, D89, D9, D90, D91, D92, D93, D94, D95, D96, D97, D98, D99: footprint LED_SMD:LED_0402_1005Metric -> LED_SMD:LED_0603_1608Metric
- U3: footprint Package_SON:Winbond_USON-8-1EP_3x2mm_P0.5mm_EP0.2x1.6mm -> Package_SO:SOIC-8_5.3x5.3mm_P1.27mm
Connections:
- net at U1.30 (GPIO19): now also J4.9 (Pin_9)
- net at U1.29 (GPIO18): now also J4.8 (Pin_8)
- net at U1.28 (GPIO17): now also J4.7 (Pin_7)
- net at U1.27 (GPIO16): now also J4.6 (Pin_6)
- net at U1.11 (GPIO8): now also J3.9 (Pin_9)
- net at U1.12 (GPIO9): now also J3.10 (Pin_10)
- net at U1.13 (GPIO10): now also J3.11 (Pin_11)
- net at U1.14 (GPIO11): now also J4.1 (Pin_1)
- net at U1.15 (GPIO12): now also J4.2 (Pin_2)
- net at U1.16 (GPIO13): now also J4.3 (Pin_3)
- net at U1.17 (GPIO14): now also J4.4 (Pin_4)
- net at U1.18 (GPIO15): now also J4.5 (Pin_5)
- net at U1.2 (GPIO0): now also J3.1 (Pin_1)
- net at U1.3 (GPIO1): now also J3.2 (Pin_2)
- net at U1.31 (GPIO20): now also J4.10 (Pin_10)
- net at U1.32 (GPIO21): now also J4.11 (Pin_11)
- net at U1.38 (GPIO26_ADC0): now also J6.1 (Pin_1)
- net at U1.39 (GPIO27_ADC1): now also J6.2 (Pin_2)
- net at U1.4 (GPIO2): now also J3.3 (Pin_3)
- net at U1.40 (GPIO28_ADC2): now also J6.3 (Pin_3)
- net at U1.41 (GPIO29_ADC3): now also J6.4 (Pin_4)
- net at U1.5 (GPIO3): now also J3.4 (Pin_4)
- net at U1.6 (GPIO4): now also J3.5 (Pin_5)
- net at U1.7 (GPIO5): now also J3.6 (Pin_6)
- net at U1.8 (GPIO6): now also J3.7 (Pin_7)
- net at U1.9 (GPIO7): now also J3.8 (Pin_8)
- no-connect marks 19 -> 1

Commit message: Add files via upload
Parts:
- removed J3, J4: Conn_01x11_Pin, Connector_PinHeader_2.54mm:PinHeader_2x06_P2.54mm_Vertical, symbol Connector:Conn_01x11_Pin
- removed J6: Conn_01x04_Socket, Connector_PinHeader_2.54mm:PinHeader_1x04_P2.54mm_Vertical, symbol Connector:Conn_01x04_Socket
- added J3: Conn_01x13_Pin, Connector_PinHeader_1.00mm:PinHeader_1x13_P1.00mm_Vertical_SMD_Pin1Left, symbol Connector:Conn_01x13_Pin
- added J4: Conn_01x06_Pin, Connector_PinHeader_1.00mm:PinHeader_1x06_P1.00mm_Vertical_SMD_Pin1Left, symbol Connector:Conn_01x06_Pin
- added J5: Conn_01x04_Pin, Connector_PinHeader_1.00mm:PinHeader_1x04_P1.00mm_Vertical_SMD_Pin1Left, symbol Connector:Conn_01x04_Pin
- added J6: Conn_01x03_Pin, Connector_PinHeader_1.00mm:PinHeader_1x03_P1.00mm_Vertical_SMD_Pin1Left, symbol Connector:Conn_01x03_Pin
- added R11: 10k, Resistor_SMD:R_0402_1005Metric, symbol Device:R
- D1, D10, D100, D101, D102, D103, D104, D105, D106, D107, D108, D109, D11, D110, D111, D112, D113, D114, D115, D116, D117, D118, D119, D12, D120, D121, D122, D123, D124, D125, D126, D127, D128, D129, D13, D130, D131, D132, D133, D134, D135, D136, D137, D138, D139, D14, D140, D141, D142, D143, D144, D15, D16, D17, D18, D19, D2, D20, D21, D22, D23, D24, D25, D26, D27, D28, D29, D3, D30, D31, D32, D33, D34, D35, D36, D37, D38, D39, D4, D40, D41, D42, D43, D44, D45, D46, D47, D48, D49, D5, D50, D51, D52, D53, D54, D55, D56, D57, D58, D59, D6, D60, D61, D62, D63, D64, D65, D66, D67, D68, D69, D7, D70, D71, D72, D73, D74, D75, D76, D77, D78, D79, D8, D80, D81, D82, D83, D84, D85, D86, D87, D88, D89, D9, D90, D91, D92, D93, D94, D95, D96, D97, D98, D99: footprint LED_SMD:LED_0603_1608Metric -> LED_SMD:LED_0402_1005Metric
Connections:
- net +3V3: now also C10.1, U1.1 (IOVDD), U1.10 (IOVDD), U1.22 (IOVDD), U1.33 (IOVDD), U1.42 (IOVDD), U1.43 (ADC_AVDD), U1.44 (VREG_IN), U1.48 (USB_VDD), U1.49 (IOVDD), R11.1; no longer R15.2, U1.56 (QSPI_SS), U3.1 (~{CS})
- net GND: no longer C10.1, U1.1 (IOVDD), U1.10 (IOVDD), U1.22 (IOVDD), U1.33 (IOVDD), U1.42 (IOVDD), U1.43 (ADC_AVDD), U1.44 (VREG_IN), U1.48 (USB_VDD), U1.49 (IOVDD)
- net at U1.11 (GPIO8): now also J3.5 (Pin_5)
- net at U1.12 (GPIO9): now also J3.4 (Pin_4)
- net at U1.13 (GPIO10): now also J3.3 (Pin_3)
- net at U1.14 (GPIO11): now also J3.2 (Pin_2)
- net at U1.15 (GPIO12): now also J3.1 (Pin_1)
- net at U1.16 (GPIO13): now also J6.3 (Pin_3)
- net at U1.17 (GPIO14): now also J6.2 (Pin_2)
- net at U1.18 (GPIO15): now also J6.1 (Pin_1)
- net at U1.2 (GPIO0): now also J3.13 (Pin_13)
- net at U1.27 (GPIO16): now also J4.6 (Pin_6)
- net at U1.28 (GPIO17): now also J4.5 (Pin_5)
- net at U1.29 (GPIO18): now also J4.4 (Pin_4)
- net at U1.3 (GPIO1): now also J3.12 (Pin_12)
- net at U1.30 (GPIO19): now also J4.3 (Pin_3)
- net at U1.31 (GPIO20): now also J4.2 (Pin_2)
- net at U1.32 (GPIO21): now also J4.1 (Pin_1)
- net at U1.38 (GPIO26_ADC0): now also J5.4 (Pin_4)
- net at U1.39 (GPIO27_ADC1): now also J5.3 (Pin_3)
- net at U1.4 (GPIO2): now also J3.11 (Pin_11)
- net at U1.40 (GPIO28_ADC2): now also J5.2 (Pin_2)
- net at U1.41 (GPIO29_ADC3): now also J5.1 (Pin_1)
- net at U1.5 (GPIO3): now also J3.10 (Pin_10)
- net at U1.6 (GPIO4): now also J3.9 (Pin_9)
- net at U1.7 (GPIO5): now also J3.8 (Pin_8)
- net at U1.8 (GPIO6): now also J3.7 (Pin_7)
- net at U1.9 (GPIO7): now also J3.6 (Pin_6)
- new net QSPI_SS: R11.2, R15.2, U1.56 (QSPI_SS), U3.1 (~{CS})
Other:
- moved on the sheet: C10
